File: PCBs/serverPCB/serverPCB.kicad_pcb (KiCad board)
At the start: 2 copper layers, 45.7 x 61 mm, 5 parts, among them J1 Screw_Terminal_01x04

Commit message: working with interrupts
Parts:
- SIMB I2C: renamed from J1
Connections:
- 10K pad 2: Net-(J1-Pin_1) -> /3V3 (x2)
- MCU pad 3V3: unconnected-(MCU1-Pad3V3) -> /3V3
Routing:
- net /3V3: track 0.00 -> 35.7 mm
- net Net-(J1-Pin_1): track 38.0 -> 27.1 mm
- net Net-(J1-Pin_3): track 16.1 -> 19.0 mm
Other:
- board text added: "CS"
- board text removed: "CS/ 3V3"
Changed lines of the file:
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@@
   (net 6 "unconnected-(MCU1-D2-Pad2)")
   (net 7 "unconnected-(MCU1-D3-Pad3)")
-  (net 8 "unconnected-(MCU1-Pad3V3)")
+  (net 8 "/3V3")
   (net 9 "unconnected-(MCU1-D4-Pad4)")
   (net 10 "unconnected-(MCU1-D5-Pad5)")
@@
     (property "ki_keywords" "screw terminal")
     (attr through_hole)
-    (fp_text reference "J1" (at 3.81 -4.16 90) (layer "F.SilkS")
-        (effects (font (size 1 1) (thickness 0.15)))
-    )
-    (fp_text value "Screw_Terminal_01x04" (at 3.81 4.16 90) (layer "F.Fab")
-        (effects (font (size 1 1) (thickness 0.15)))
-    )
-    (fp_text user "${REFERENCE}" (at 3.81 2 90) (layer "F.Fab")
+    (fp_text reference "SIMB I2C" (at 3.81 -4.16 90) (layer "F.SilkS")
+        (effects (font (size 1 1) (thickness 0.15)))
+    )
+    (fp_text value "Screw_Terminal_01x04" (at 0 12.7 90) (layer "F.Fab") hide
         (effects (font (size 1 1) (thickness 0.15)))
     )
@@
         (effects (font (size 1 1) (thickness 0.15)))
     )
-    (fp_text value "10K" (at 3.81 2.37 90) (layer "F.Fab")
-        (effects (font (size 1 1) (thickness 0.15)))
-    )
-    (fp_text user "${REFERENCE}" (at 3.81 0 90) (layer "F.Fab")
+    (fp_text value "10K" (at 3.81 2.37 90) (layer "F.Fab") hide
         (effects (font (size 1 1) (thickness 0.15)))
     )
@@
       (net 1 "Net-(J1-Pin_2)") (pintype "passive"))
     (pad "2" thru_hole oval (at 7.62 0 90) (size 1.6 1.6) (drill 0.8) (layers "*.Cu" "*.Mask")
-      (net 38 "Net-(J1-Pin_1)") (pintype "passive"))
+      (net 8 "/3V3") (pintype "passive"))
     (model "${KICAD6_3DMODEL_DIR}/Resistor_THT.3dshapes/R_Axial_DIN0207_L6.3mm_D2.5mm_P7.62mm_Horizontal.wrl"
       (offset (xyz 0 0 0))
@@
         (effects (font (size 1 1) (thickness 0.15)))
     )
-    (fp_text value "10K" (at 3.81 2.37 90) (layer "F.Fab")
-        (effects (font (size 1 1) (thickness 0.15)))
-    )
-    (fp_text user "${REFERENCE}" (at 3.81 0 90) (layer "F.Fab")
+    (fp_text value "10K" (at 3.81 2.37 90) (layer "F.Fab") hide
         (effects (font (size 1 1) (thickness 0.15)))
     )
@@
       (net 2 "Net-(J1-Pin_3)") (pintype "passive"))
     (pad "2" thru_hole oval (at 7.62 0 90) (size 1.6 1.6) (drill 0.8) (layers "*.Cu" "*.Mask")
-      (net 38 "Net-(J1-Pin_1)") (pintype "passive"))
+      (net 8 "/3V3") (pintype "passive"))
     (model "${KICAD6_3DMODEL_DIR}/Resistor_THT.3dshapes/R_Axial_DIN0207_L6.3mm_D2.5mm_P7.62mm_Horizontal.wrl"
       (offset (xyz 0 0 0))
@@
       (net 7 "unconnected-(MCU1-D3-Pad3)") (pinfunction "D3") (pintype "bidirectional+no_connect"))
     (pad "3V3" thru_hole circle (at -12.7 7.62) (size 1.524 1.524) (drill 0.9) (layers "*.Cu" "*.Mask")
-      (net 8 "unconnected-(MCU1-Pad3V3)") (pinfunction "3V3") (pintype "power_out+no_connect"))
+      (net 8 "/3V3") (pinfunction "3V3") (pintype "power_out"))
     (pad "4" thru_hole circle (at 10.16 -5.08) (size 1.524 1.524) (drill 0.9) (layers "*.Cu" "*.Mask")
       (net 9 "unconnected-(MCU1-D4-Pad4)") (pinfunction "D4") (pintype "bidirectional+no_connect"))
@@
     (effects (font (size 1 1) (thickness 0.15)))
   )
-  (gr_text "CS/\n3V3" (at 160.02 116.84) (layer "F.SilkS")
+  (gr_text "CS" (at 160.02 116.84) (layer "F.SilkS")
     (effects (font (size 1 1) (thickness 0.15)))
   )
-  (segment (start 154.94 114.3) (end 148.76 114.3) (width 0.25) (layer "F.Cu") (net 1))
-  (segment (start 148.76 114.3) (end 146.22 116.84) (width 0.25) (layer "F.Cu") (net 1))
-  (segment (start 157.48 111.76) (end 154.94 114.3) (width 0.25) (layer "F.Cu") (net 1))
-  (segment (start 157.48 105.41) (end 157.48 111.76) (width 0.25) (layer "F.Cu") (net 1))
-  (segment (start 148.76 111.76) (end 146.22 114.3) (width 0.25) (layer "F.Cu") (net 2))
-  (segment (start 152.4 105.41) (end 152.4 111.76) (width 0.25) (layer "F.Cu") (net 2))
-  (segment (start 154.94 111.76) (end 148.76 111.76) (width 0.25) (layer "F.Cu") (net 2))
+  (segment (start 148.76 114.3) (end 146.22 116.84) (width 0.25) (layer "B.Cu") (net 1))
+  (segment (start 157.48 105.41) (end 157.48 111.76) (width 0.25) (layer "B.Cu") (net 1))
+  (segment (start 157.48 111.76) (end 154.94 114.3) (width 0.25) (layer "B.Cu") (net 1))
+  (segment (start 154.94 114.3) (end 148.76 114.3) (width 0.25) (layer "B.Cu") (net 1))
+  (segment (start 152.4 105.41) (end 153.53137 105.41) (width 0.25) (layer "B.Cu") (net 2))
+  (segment (start 156.365 108.24363) (end 156.365 110.335) (width 0.25) (layer "B.Cu") (net 2))
+  (segment (start 153.53137 105.41) (end 156.365 108.24363) (width 0.25) (layer "B.Cu") (net 2))
+  (segment (start 156.365 110.335) (end 154.94 111.76) (width 0.25) (layer "B.Cu") (net 2))
+  (segment (start 154.94 111.76) (end 148.76 111.76) (width 0.25) (layer "B.Cu") (net 2))
+  (segment (start 148.76 111.76) (end 146.22 114.3) (width 0.25) (layer "B.Cu") (net 2))
   (segment (start 153.840001 110.319999) (end 124.800001 110.319999) (width 0.25) (layer "B.Cu") (net 3))
   (segment (start 126 71.12) (end 123.36 71.12) (width 0.25) (layer "B.Cu") (net 3))
@@
   (segment (start 131.08 66.04) (end 126 71.12) (width 0.25) (layer "B.Cu") (net 3))
   (segment (start 124.800001 110.319999) (end 123.36 111.76) (width 0.25) (layer "B.Cu") (net 3))
-  (segment (start 141.24 66.04) (end 141.24 100.6) (width 0.25) (layer "B.Cu") (net 15))
+  (segment (start 152.4 97.79) (end 127.17 97.79) (width 0.25) (layer "B.Cu") (net 8))
+  (segment (start 127.17 97.79) (end 123.36 101.6) (width 0.25) (layer "B.Cu") (net 8))
+  (segment (start 157.48 97.79) (end 152.4 97.79) (width 0.25) (layer "B.Cu") (net 8))
+  (segment (start 141.24 66.04) (end 141.24 100.6) (width 0.25) (layer "F.Cu") (net 15))
+  (segment (start 144.78 104.14) (end 146.22 104.14) (width 0.25) (layer "F.Cu") (net 15))
+  (segment (start 141.24 100.6) (end 144.78 104.14) (width 0.25) (layer "F.Cu") (net 15))
   (segment (start 140.153 64.953) (end 129.627 64.953) (width 0.25) (layer "B.Cu") (net 15))
   (segment (start 141.24 66.04) (end 140.153 64.953) (width 0.25) (layer "B.Cu") (net 15))
-  (segment (start 144.78 104.14) (end 146.22 104.14) (width 0.25) (layer "B.Cu") (net 15))
   (segment (start 129.627 64.953) (end 128.54 66.04) (width 0.25) (layer "B.Cu") (net 15))
-  (segment (start 141.24 100.6) (end 144.78 104.14) (width 0.25) (layer "B.Cu") (net 15))
   (segment (start 136.16 83.72) (end 123.36 96.52) (width 0.25) (layer "B.Cu") (net 25))
   (segment (start 136.16 66.04) (end 136.16 83.72) (width 0.25) (layer "B.Cu") (net 25))
@@
   (segment (start 133.62 83.72) (end 123.36 93.98) (width 0.25) (layer "B.Cu") (net 27))
   (segment (start 133.62 66.04) (end 133.62 83.72) (width 0.25) (layer "B.Cu") (net 27))
-  (segment (start 146.22 93.98) (end 148.59 93.98) (width 0.25) (layer "F.Cu") (net 38))
-  (segment (start 160.02 100.33) (end 160.02 116.84) (width 0.25) (layer "F.Cu") (net 38))
-  (segment (start 160.02 116.84) (end 154.94 116.84) (width 0.25) (layer "F.Cu") (net 38))
-  (segment (start 152.4 97.79) (end 157.48 97.79) (width 0.25) (layer "F.Cu") (net 38))
-  (segment (start 157.48 97.79) (end 160.02 100.33) (width 0.25) (layer "F.Cu") (net 38))
-  (segment (start 148.59 93.98) (end 152.4 97.79) (width 0.25) (layer "F.Cu") (net 38))
+  (segment (start 149.86 96.52) (end 147.32 93.98) (width 0.25) (layer "F.Cu") (net 38))
+  (segment (start 154.94 116.84) (end 149.86 111.76) (width 0.25) (layer "F.Cu") (net 38))
+  (segment (start 149.86 111.76) (end 149.86 96.52) (width 0.25) (layer "F.Cu") (net 38))
+  (segment (start 147.32 93.98) (end 146.22 93.98) (width 0.25) (layer "F.Cu") (net 38))
 )

Commit message: pcb edits
Parts:
- removed 10K (x2): 10K, Resistor_THT:R_Axial_DIN0207_L6.3mm_D2.5mm_P7.62mm_Horizontal
- added C1: 10µF, Capacitor_THT:CP_Radial_Tantal_D4.5mm_P2.50mm, F.Cu at (161.3, 82.5)
- added C2: 47µF, Capacitor_THT:CP_Radial_Tantal_D4.5mm_P2.50mm, F.Cu at (161.3, 77.5)
- added C3: 47µF, Capacitor_THT:CP_Radial_Tantal_D4.5mm_P2.50mm, F.Cu at (161.3, 72.4)
- added G***: LOGO, LOGO, F.Cu at (154.9, 64.3)
- added U1: TPSM84203, Converter_DCDC:Pololu_D24V5F9, F.Cu at (154.9, 77.7)
- added U2: ~, Converter_DCDC:Pololu_logicLevelShifter, F.Cu at (154.9, 91.4)
- J1: renamed from SIMB I2C; footprint TerminalBlock_Phoenix:TerminalBlock_Phoenix_MPT-0,5-4-2.54_1x04_P2.54mm_Horizontal -> TerminalBlock_Phoenix:TerminalBlock_Phoenix_MPT-0,5-5-2.54_1x05_P2.54mm_Horizontal
- moved µSD 1.13 mm to (134.6, 79.8)
Connections:
- J1 pad 4: /GND -> Net-(J1-Pin_4)
- MCU pad 20: Net-(J1-Pin_2) -> Net-(MCU1-SDA)
- MCU pad 21: Net-(J1-Pin_3) -> Net-(MCU1-SCL)
- MCU pad 5V: unconnected-(MCU1-Pad5V) -> /5V
- MCU pad 6: Net-(J1-Pin_1) -> Net-(MCU1-D6)
- MCU pad VIN: unconnected-(MCU1-PadVIN) -> Net-(U1-Vout)
- µSD pad 7: /sd_cs -> /3V3
Routing:
- net /GND: track 42.5 -> 125.8 mm
- net Net-(U1-Vout): track 0.00 -> 65.0 mm
- net /5V: track 0.00 -> 47.8 mm
- net /3V3: track 35.7 -> 73.2 mm
- net Net-(MCU1-SDA): track 0.00 -> 27.4 mm
- net Net-(MCU1-SCL): track 0.00 -> 27.4 mm
- net Net-(J1-Pin_1): track 27.1 -> 49.7 mm
- net Net-(J1-Pin_4): track 0.00 -> 21.9 mm
- net /sd_cs: track 54.6 -> 41.1 mm
- net Net-(MCU1-D6): track 0.00 -> 4.91 mm
- net Net-(J1-Pin_2): track 19.7 -> 22.8 mm
- net Net-(J1-Pin_3): track 19.0 -> 21.9 mm
Other:
- board size 45.7 x 61 mm -> 53.3 x 66 mm
- board text added: "5V"
- board text added: "< 18V"
- board text added: "< GND"
- board text added: "< SCL"
- board text added: "< SC_CS"
- board text added: "<> SDA"
- board text added: "D24V5F6"
- board text added: "HV"
- board text added: "LV"
- board text added: "NC"
- board text added: "SCL^"
- board text added: "SC_CS^"
- board text added: "SDA^"
- board text added: "SnowTATOS server v1.0 May 14 2023"
- board text added: "Vin"
- board text added: "Vout"
- board text added: "ian.a.raphael.th@dartmouth.edu Thayer School of Engineering Dartmouth College"
- board text removed: "CS"
- board text removed: "SCA"
- board text removed: "SDA"
