File: PCBs/serverPCB/serverPCB.kicad_sch (KiCad schematic)
At the start: 5 parts, among them J1 Screw_Terminal_01x04

Commit message: working with interrupts
Connections:
- net at J1.1 (Pin_1), MCU1.6 (D6): no longer R1.2, R2.2
- net 3V3: now reaches MCU1.3V3
- net 3V3: now also R1.2, R2.2
- no-connect marks 31 -> 30
Other:
- note added: "CS"
- note added: "GND"
- note added: "SCA"
- note added: "SDA"
- note added: "simb i2c screw header"
- note removed: "i2c (simb) header"
- moved on the sheet: R1, R2

Commit message: pcb edits
Parts:
- removed R1, R2: 10K, Resistor_THT:R_Axial_DIN0207_L6.3mm_D2.5mm_P7.62mm_Horizontal, symbol Device:R
- added C1: 10µF, Capacitor_THT:CP_Radial_Tantal_D4.5mm_P2.50mm, symbol Device:C
- added C2, C3: 47µF, Capacitor_THT:CP_Radial_Tantal_D4.5mm_P2.50mm, symbol Device:C
- added U1: TPSM84203, Converter_DCDC:Pololu_D24V5F9, symbol Regulator_Switching:Pololu_D24V5F9
- added U2: ~, Converter_DCDC:Pololu_logicLevelShifter, symbol Logic_LevelTranslator:Pololu_logicLevelShifter
- J1: footprint TerminalBlock_Phoenix:TerminalBlock_Phoenix_MPT-0,5-4-2.54_1x04_P2.54mm_Horizontal -> TerminalBlock_Phoenix:TerminalBlock_Phoenix_MPT-0,5-5-2.54_1x05_P2.54mm_Horizontal; symbol Connector:Screw_Terminal_01x04 -> Connector:Screw_Terminal_01x05
Connections:
- net 3V3: now also µSD1.7 (3V3), U2.1 (LV)
- net GND: now also J1.5 (Pin_5), C1.2, C2.2, C3.2, U1.3 (GND); no longer J1.4 (Pin_4)
- net sd_cs: no longer µSD1.7 (3V3)
- net at J1.1 (Pin_1): now also C1.1, U1.2 (Vin); no longer MCU1.6 (D6)
- net at J1.2 (Pin_2): now also U2.9 (H3); no longer MCU1.20 (SDA)
- net at J1.3 (Pin_3): now also U2.8 (H2); no longer MCU1.21 (SCL)
- net 5V: now reaches MCU1.5V
- net 5V: now also U2.6 (HV)
- net at MCU1.VIN: now also C2.1, C3.1, U1.4 (Vout)
- new net: J1.4 (Pin_4), U2.7 (H1)
- new net: MCU1.20 (SDA), U2.3 (L2)
- new net: MCU1.21 (SCL), U2.2 (L1)
- new net: MCU1.6 (D6), U2.4 (L3)
- no-connect marks 30 -> 31
Other:
- note added: "SCL"
- note added: "SC_CS"
- note added: "Vin (18V)"
- note added: "simb screw header"
- note removed: "CS"
- note removed: "SCA"
- note removed: "i2c pullups"
- note removed: "simb i2c screw header"
