File: PCBs/tempLogger_clientPCB/tempLogger_clientPCB.kicad_sch (KiCad schematic)
At the start: 5 parts

Commit message: mostly pcb updates. beginning of arcwatch deployment code. updates to libs
Parts:
- added BT1, BT2: 3.6V, Battery:battery_c_cell_solderTabs, symbol Device:Battery
- added C1: 10µF, Capacitor_THT:CP_Radial_Tantal_D4.5mm_P2.50mm, symbol Device:C
- added C2, C3: 47µF, Capacitor_THT:CP_Radial_Tantal_D4.5mm_P2.50mm, symbol Device:C
- added D1: 1n5820, Diode_THT:D_DO-41_SOD81_P10.16mm_Horizontal, symbol Diode:1N5817
- added JST1: JST male flying leads, TestPoint:TestPoint_2Pads_Pitch5.08mm_Drill1.3mm, symbol Connector_Generic:Conn_01x02
- added U1: TPSM84203, Converter_DCDC:Converter_DCDC_TRACO_TSR-1_THT, symbol Regulator_Switching:TSR_1-2433
- SnowPinger1: renamed from SnowPinger; footprint TerminalBlock_Phoenix:TerminalBlock_Phoenix_MPT-0,5-3-2.54_1x03_P2.54mm_Horizontal -> TerminalBlock_TE-Connectivity:TerminalBlock_TE_282834-3_1x03_P2.54mm_Horizontal
- renumbered MCU to MCU1
Connections:
- net 3V3: now also µSD1.7 (3V3)
- net GND: now also BT1.2 (-), C1.2, C2.2, C3.2, JST1.2 (Pin_2), U1.2 (GND)
- net sd_cs: no longer µSD1.7 (3V3)
- new net: BT2.1 (+), C1.1, U1.1 (Vin)
- new net: BT1.1 (+), BT2.2 (-)
- new net: C2.1, C3.1, D1.2 (A), U1.3 (Vout)
- new net: D1.1 (K), JST1.1 (Pin_1)

Commit message: pcb edits
Parts:
- removed C1: 10µF, Capacitor_THT:CP_Radial_Tantal_D4.5mm_P2.50mm, symbol Device:C
- removed C2, C3: 47µF, Capacitor_THT:CP_Radial_Tantal_D4.5mm_P2.50mm, symbol Device:C
- removed D1: 1n5820, Diode_THT:D_DO-41_SOD81_P10.16mm_Horizontal, symbol Diode:1N5817
- removed JST1: JST male flying leads, TestPoint:TestPoint_2Pads_Pitch5.08mm_Drill1.3mm, symbol Connector_Generic:Conn_01x02
- removed SnowPinger1: Screw_Terminal_01x03, TerminalBlock_TE-Connectivity:TerminalBlock_TE_282834-3_1x03_P2.54mm_Horizontal, symbol Connector:Screw_Terminal_01x03
- removed U1: TPSM84203, Converter_DCDC:Converter_DCDC_TRACO_TSR-1_THT, symbol Regulator_Switching:TSR_1-2433
- renumbered DS18B20 to Pinger/Temp
Connections:
- net at BT2.1 (+): now also MCU1.VIN
- net at MCU1.8 (D8), Pinger/Temp.4 (Pin_4), R1.1: no longer Pinger/Temp.1 (Pin_1)
- net at MCU1.7 (D7), Pinger/Temp.5 (Pin_5), R1.2: no longer Pinger/Temp.2 (Pin_2)
- net at MCU1.0 (SERIAL1_RX): now also Pinger/Temp.2 (Pin_2)
- net at MCU1.11 (D11): now also Pinger/Temp.1 (Pin_1)
- no-connect marks 28 -> 27
Other:
- note removed: "Snow pinger header"
- note removed: "Temperature sensor header"
- moved on the sheet: BT1, BT2
