File: PCBs/V2/tempLogger_clientPCB_2xBattHolder/tempLogger_clientPCB_2xBattHolder.kicad_sch (KiCad schematic)
At the start: 5 parts

Commit message: fixed pinger read error
Parts:
- removed U1: ~, Battery:BatteryHolder_Keystone_2233, symbol Device:keystone_2233_D_cell_2Batt_holder
- added U1: keystone_2233_D_cell_4Batt_holder, Battery:BatteryHolder_Keystone_2233_4Cell, symbol Device:keystone_2233_D_cell_4Batt_holder
Connections:
- net GND: now also U1.0
- net VBAT: now also U1.1
Changed lines of the file:
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@@
   (junction (at 160.02 85.09) (diameter 0) (color 0 0 0 0)
   )
-  (wire (pts (xy 124.46 106.68) (xy 124.46 110.49))
-    (stroke (width 0) (type default))
-  )
   (wire (pts (xy 146.05 63.5) (xy 171.45 63.5))
     (stroke (width 0) (type default))
@@
     (stroke (width 0) (type default))
   )
-  (wire (pts (xy 149.86 171.45) (xy 149.86 175.26))
-    (stroke (width 0) (type default))
-  )
   (wire (pts (xy 129.54 73.66) (xy 129.54 58.42))
     (stroke (width 0) (type default))
   )
-  (wire (pts (xy 124.46 171.45) (xy 124.46 139.7))
-    (stroke (width 0) (type default))
-  )
   (wire (pts (xy 168.91 90.17) (xy 171.45 90.17))
     (stroke (width 0) (type default))
@@
     (stroke (width 0) (type default))
   )
+  (wire (pts (xy 120.65 118.11) (xy 120.65 124.46))
+    (stroke (width 0) (type default))
+  )
   (wire (pts (xy 147.32 73.66) (xy 167.64 73.66))
     (stroke (width 0) (type default))
   )
-  (wire (pts (xy 124.46 139.7) (xy 149.86 139.7))
+  (wire (pts (xy 146.05 118.11) (xy 146.05 124.46))
     (stroke (width 0) (type default))
   )
@@
     (stroke (width 0) (type default))
   )
-  (wire (pts (xy 149.86 139.7) (xy 149.86 110.49))
-    (stroke (width 0) (type default))
-  )
   (wire (pts (xy 171.45 87.63) (xy 160.02 87.63))
     (stroke (width 0) (type default))
@@
     (effects (font (size 1.27 1.27)) (justify left bottom))
   )
-  (label "VBAT" (at 149.86 175.26 270) (fields_autoplaced)
-    (effects (font (size 1.27 1.27)) (justify right bottom))
+  (label "VBAT" (at 146.05 118.11 90) (fields_autoplaced)
+    (effects (font (size 1.27 1.27)) (justify left bottom))
   )
   (label "RXD1" (at 146.05 57.15 180) (fields_autoplaced)
     (effects (font (size 1.27 1.27)) (justify right bottom))
   )
-  (label "GND" (at 124.46 106.68 90) (fields_autoplaced)
+  (label "GND" (at 120.65 118.11 90) (fields_autoplaced)
     (effects (font (size 1.27 1.27)) (justify left bottom))
   )
@@
     (pin "VIN")
     (instances
-      (project "tempLogger_clientPCB"
+      (project "tempLogger_clientPCB_2xBattHolder"
         (path "/e9a5d9db-8c3f-49ab-905c-e4478fcc15ff"
           (reference "MCU2") (unit 1)
@@
     (pin "3")
     (instances
-      (project "tempLogger_clientPCB"
+      (project "tempLogger_clientPCB_2xBattHolder"
         (path "/e9a5d9db-8c3f-49ab-905c-e4478fcc15ff"
           (reference "Temp1") (unit 1)
@@
     (pin "3")
     (instances
-      (project "tempLogger_clientPCB"
+      (project "tempLogger_clientPCB_2xBattHolder"
         (path "/e9a5d9db-8c3f-49ab-905c-e4478fcc15ff"
           (reference "Pinger1") (unit 1)
@@
     )
   )
-  (symbol (lib_id "Device:keystone_2233_D_cell_2Batt_holder") (at 137.16 140.97 0) (mirror y) (unit 1)
-    (in_bom yes) (on_board yes) (dnp no)
-    (property "Reference" "U1" (at 110.49 141.605 0)
-      (effects (font (size 1.27 1.27)) (justify left))
-    )
-    (property "Value" "~" (at 137.16 140.97 0)
-      (effects (font (size 1.27 1.27)))
-    )
-    (property "Footprint" "Battery:BatteryHolder_Keystone_2233" (at 137.16 140.97 0)
-      (effects (font (size 1.27 1.27)) hide)
-    )
-    (property "Datasheet" "" (at 137.16 140.97 0)
+  (symbol (lib_id "Device:keystone_2233_D_cell_4Batt_holder") (at 133.35 154.94 0) (unit 1)
+    (in_bom yes) (on_board yes) (dnp no) (fields_autoplaced)
+    (property "Reference" "U1" (at 160.02 153.035 0)
+      (effects (font (size 1.27 1.27)) (justify left))
+    )
+    (property "Value" "keystone_2233_D_cell_4Batt_holder" (at 160.02 155.575 0)
+      (effects (font (size 1.27 1.27)) (justify left))
+    )
+    (property "Footprint" "Battery:BatteryHolder_Keystone_2233_4Cell" (at 133.35 154.94 0)
+      (effects (font (size 1.27 1.27)) hide)
+    )
+    (property "Datasheet" "" (at 133.35 154.94 0)
       (effects (font (size 1.27 1.27)) hide)
     )
     (pin "0")
     (pin "1")
-    (pin "2")
-    (pin "3")
-    (instances
-      (project "tempLogger_clientPCB"
+    (instances
+      (project "tempLogger_clientPCB_2xBattHolder"
         (path "/e9a5d9db-8c3f-49ab-905c-e4478fcc15ff"
           (reference "U1") (unit 1)
@@
     (pin "2")
     (instances
-      (project "tempLogger_clientPCB"
+      (project "tempLogger_clientPCB_2xBattHolder"
         (path "/e9a5d9db-8c3f-49ab-905c-e4478fcc15ff"
           (reference "R1") (unit 1)
